Commit message: added trees into bullet and added modified files

File: models/tree1.urdf (robot description, URDF)
Before this commit: robot tree1, 1 links, 0 joints
Links:
- link base_link: geometry collision mesh filename=package://sherpa_spatial_relations/models/tree2.stl; visual mesh filename=package://sherpa_spatial_relations/models/tree1.stl

Commit message: added new files

File: models/tree1.urdf (robot description, URDF)
Before this commit: robot tree1, 1 links, 0 joints
Links:
- link base_link: mass None -> 1; geometry visual mesh filename=package://sherpa_spatial_relations/models/tree_col-6.dae
